File: hardware/gambos-pcb.kicad_pcb (KiCad board)
At the start: 4 copper layers, 75.9 x 58.3 mm, 130 parts, among them J1 JST-PH, J10 Conn_01x03_Pin, J11 Conn_01x03_Pin, J12 Conn_01x03_Pin, J13 Conn_01x03_Pin, J2 Micro_SD_Card, J4 FTSH-105-01-F-DV-K-A, J5 Conn_01x03_Pin, J7 Conn_01x03_Pin, J9 Conn_01x03_Pin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

Commit message: Docker environment fixes
Changed lines of the file:
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@@
 			(pdf_back_fp_property_popups yes)
 			(pdf_metadata yes)
-			(pdf_single_document no)
+			(pdf_single_document yes)
 			(dxfpolygonmode yes)
 			(dxfimperialunits yes)
@@
 			(psnegative no)
 			(psa4output no)
-			(plot_black_and_white yes)
+			(plot_black_and_white no)
 			(sketchpadsonfab no)
 			(plotpadnumbers no)
@@
 			(crossoutdnponfab yes)
 			(subtractmaskfromsilk no)
-			(outputformat 1)
+			(outputformat 4)
 			(mirror no)
 			(drillshape 0)
 			(scaleselection 1)
-			(outputdirectory "C:/Projects/gambos/hardware/gerbers/")
+			(outputdirectory "/home/mikael/gambos/hardware/Gambos-Flight-Controller/")
 		)
 	)
@@
 			(at 0 7.46 0)
 			(layer "F.Fab")
+			(hide yes)
 			(effects
 				(font
@@
 		(tags "capacitor")
 		(property "Reference" "C13"
-			(at -0.830002 3.21 0)
+			(at -0.530002 3.01 0)
 			(layer "F.SilkS")
 			(effects
@@
 		(tags "resistor")
 		(property "Reference" "R3"
-			(at 0 1.43 0)
+			(at 2.42 0.1 0)
 			(layer "B.SilkS")
-			(hide yes)
 			(effects
 				(font
@@
 		(tags "capacitor")
 		(property "Reference" "C20"
-			(at 0 1.43 90)
+			(at 2.87 0.041667 90)
 			(layer "B.SilkS")
-			(hide yes)
 			(effects
 				(font
@@
 		(tags "capacitor")
 		(property "Reference" "C4"
-			(at -1.81 2.25 90)
+			(at -0.05 1.7 0)
 			(layer "B.SilkS")
 			(effects
@@
 		(tags "capacitor")
 		(property "Reference" "C31"
-			(at 0 1.43 90)
+			(at 2.77 0.1 90)
 			(layer "B.SilkS")
-			(hide yes)
 			(effects
 				(font
@@
 		(tags "capacitor")
 		(property "Reference" "C15"
-			(at 0 1.43 90)
+			(at 2.87 -0.001667 90)
 			(layer "B.SilkS")
-			(hide yes)
 			(effects
 				(font
@@
 			(at 0.145 1.48 90)
 			(layer "B.SilkS")
-			(hide yes)
 			(effects
 				(font
@@
 		(tags "capacitor")
 		(property "Reference" "C12"
-			(at 0 1.43 90)
+			(at 2.87 -0.045 90)
 			(layer "B.SilkS")
-			(hide yes)
 			(effects
 				(font
@@
 			(at 0 1.43 0)
 			(layer "B.SilkS")
-			(hide yes)
 			(effects
 				(font
@@
 	)
 	(via
-		(at 125.75 98.51)
+		(at 125.9 98.4)
 		(size 0.6)
 		(drill 0.3)
@@
 		(polygon
 			(pts
-				(xy 125.85 101.516274) (xy 130.850003 96.45) (xy 136.1 96.45) (xy 137.6 94.95) (xy 142.725 94.95)
-				(xy 143.1 95.325) (xy 143.1 97.79375) (xy 142.44375 98.45) (xy 140.88125 98.45) (xy 140.35 98.98125)
-				(xy 140.35 99.575) (xy 139.975 99.95) (xy 138.13125 99.95) (xy 137.35 100.73125) (xy 137.35 106.3)
-				(xy 133.35 106.358588) (xy 133.35 105.535937) (xy 132.514063 104.7) (xy 130.1 104.7) (xy 129.35 105.45)
-				(xy 129.4 107) (xy 125.85 106.965625)
+				(xy 125.85 101.516274) (xy 130.850003 96.45) (xy 136.1 96.45) (xy 137.6 94.95) (xy 143 94.95) (xy 143 97.400002)
+				(xy 142.150002 98.25) (xy 140.850002 98.25) (xy 140.35 98.750002) (xy 140.35 99.35) (xy 139.75 99.95)
+				(xy 138.13125 99.95) (xy 137.35 100.73125) (xy 137.35 106.3) (xy 133.35 106.358588) (xy 133.35 105.535937)
+				(xy 132.333381 104.1) (xy 130.277118 104.1) (xy 129.35 105.45) (xy 129.4 107) (xy 125.85 106.965625)
 			)
 		)
