File: hardware/sensors_and_flash.kicad_sch (KiCad schematic)
At the start: 29 parts, among them J2 Micro_SD_Card, U2 AT25SF128A-SHB-T, U4 LSM6DSVTR, U5 BMP384, U8 IIS2MDCTR

Commit message: Docker environment fixes
Other:
- note added: "Pressure and temperature"
- note removed: "Pressure and humidity"
Changed lines of the file:
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@@
 		)
 	)
-	(text "Pressure and humidity"
+	(text "Pressure and temperature"
 		(exclude_from_sim no)
 		(at 144.526 81.788 0)
