File: hardware/MCU.kicad_sch (KiCad schematic)
At the start: 18 parts, among them U1 NRF24L01_Breakout

Commit message: Added partial documentation about the project
Other:
- moved on the sheet: C1, C2, C33, C4, C5, C6, C7, C8, C9, FB1
