File: hardware/microcontroller.kicad_sch (KiCad schematic)
At the start: 48 parts, among them J4 FTSH-105-01-F-DV-K-A, J5 Conn_01x03_Pin, SW1 SW_Push, SW3 SW_Push, U12 CM1293A-04SO, U13 CM1293A-04SO, U7 STM32F446RET6, Y2 TSX-3225_26MHZ

Commit message: Added partial documentation about the project
Other:
- moved on the sheet: C10, R30, SW3, U12
